Commit message: feat: Add urdf description and test launch file for epick gripper

File: robotiq_epick_visualization/urdf/robotiq_epick_model_macro.xacro (robot description, xacro)
@@ -1,5 +1,5 @@
 <?xml version="1.0"?>
 <robot xmlns:xacro="http://www.ros.org/wiki/xacro">
-  <xacro:include filename="$(find robotiq_epick_gripper_visualization)/urdf/robotiq_epick/robotiq_epick.gazebo.xacro"/>
+  <xacro:include filename="$(find robotiq_epick_visualization)/urdf/robotiq_epick.gazebo.xacro"/>
   <xacro:property name="joint_lower_limit" value="0.0" />
   <xacro:property name="joint_upper_limit" value="0.055" />
@@ -14,5 +14,5 @@
         <origin xyz="0 0 0.095" rpy="0 0 0"/>
         <geometry>
-          <mesh filename="package://robotiq_epick_gripper_visualization/meshes/visual/robotiq_epick.dae" scale="0.001 0.001 0.001"/>
+          <mesh filename="package://robotiq_epick_visualization/meshes/visual/robotiq_epick.dae" scale="0.001 0.001 0.001"/>
         </geometry>
         <material name="">

Commit message: feat: Add launch file to start server and driver epick gripper!

File: robotiq_epick_visualization/urdf/robotiq_epick_model_macro.xacro (robot description, xacro)
@@ -21,7 +21,7 @@
       </visual>
       <visual>
-        <origin xyz="0 0 ${0.008+0.095}" rpy="0 0 0"/>
+        <origin xyz="0 0 ${0.015+0.095}" rpy="0 0 0"/>
         <geometry>
-          <cylinder radius="0.006" length="0.016"/>
+          <cylinder radius="0.006" length="0.03"/>
         </geometry>
         <material name="">
@@ -31,7 +31,7 @@
       <collision>
         <!-- -0.095 + 0.102/2 = -0.044-->
-        <origin xyz="0 0 ${-0.044+0.095}" rpy="0 0 0"/>
+        <origin xyz="0 0 ${-0.044+0.095+0.014}" rpy="0 0 0"/>
         <geometry>
-          <cylinder radius="0.044" length="0.102"/>
+          <cylinder radius="0.044" length="0.13"/>
         </geometry>
       </collision>
@@ -49,5 +49,5 @@
       <parent link="${hand_link_name}"/>
       <child link="epick_end_effector"/>
-      <origin xyz="0 0 ${0.017+0.095}" rpy="0 0 0"/>
+      <origin xyz="0 0 ${0.13}" rpy="0 0 0"/>
     </joint>
     <link name="epick_end_effector">
@@ -56,5 +56,5 @@
         <origin rpy="0 0 0.005" xyz="0 0 0"/>
         <geometry>
-          <cylinder radius="0.024" length="0.005"/>
+          <cylinder radius="0.0225" length="0.01"/>
         </geometry>
         <!-- <material name="transparent">
